File: KiCad/Mouse_Project.kicad_pcb (KiCad board)
At the start: 2 copper layers, 1 part

Commit message: backup
Parts:
- removed REF**: NRF52840_ProMicro, 1_Custom_Library:NRF52840_ProMicro
- added J1: B2B-PH-K-S, B2B-PH-K-S:CONN2_B2B-PH-K-S_JST, F.Cu at (164.0, 87.5)
- added J2: B2B-PH-K-S_simple, B2B-PH-K-S:CONN2_B2B-PH-K-S_JST, F.Cu at (147.0, 91.0)
- added Kailh_Switch1: ~, Kailh_Switch:Kailh_Switch, F.Cu at (145.7, 74.3)
- added Kailh_Switch2: ~, Kailh_Switch:Kailh_Switch, F.Cu at (152.6, 74.3)
- added NRF52840_ProMicro1: ~, nrf52840_promicro:nrf52840_promicro, F.Cu at (88.8, 89.8)
- added PMW3389DM-T3QU1: ~, pmw3389dm-t3qu:pmw3389dm-t3qu, F.Cu at (135.6, 76.0)

Commit message: Almost done
Parts:
- removed J2: B2B-PH-K-S_simple, B2B-PH-K-S:CONN2_B2B-PH-K-S_JST
- added C1: 10uF, CL21A106KOQNNNE:CAP_CL21_SAM, B.Cu at (105.5, 111.4)
- added C10: 120pF, GRM0335C1H121JA01D:G-033_MUR, F.Cu at (101.1, 124.2)
- added C11: 10uF, CL21A106KOQNNNE:CAP_CL21_SAM, F.Cu at (98.7, 117.2)
- added C12: 0.1uF, CL10B104KB8NNNC:CAP_CL10_SAM, F.Cu at (126.3, 68.5)
- added C13: 0.1uF, CL10B104KB8NNNC:CAP_CL10_SAM, F.Cu at (120.2, 90.8)
- added C14: 0.1uF, CL10B104KB8NNNC:CAP_CL10_SAM, B.Cu at (102.2, 59.2)
- added C15: 0.1uF, CL10B104KB8NNNC:CAP_CL10_SAM, B.Cu at (127.8, 59.2)
- added C16: 0.1uF, CL10B104KB8NNNC:CAP_CL10_SAM, B.Cu at (97.2, 84.2)
- added C17: 0.1uF, CL10B104KB8NNNC:CAP_CL10_SAM, B.Cu at (97.2, 97.7)
- added C2: 4.7uF/10V, CL10A475KP8NNNC:CAP_0603_CL10A_1P6XP8_SAM, B.Cu at (105.5, 106.2)
- added C3: 0.1uF, CL10B104KB8NNNC:CAP_CL10_SAM, B.Cu at (107.2, 111.3)
- added C4: 0.1uF, CL10B104KB8NNNC:CAP_CL10_SAM, B.Cu at (107.2, 106.2)
- added C5: 0.1uF, CL10B104KB8NNNC:CAP_CL10_SAM, F.Cu at (107.2, 109.5)
- added C6: 10uF, CL21A106KOQNNNE:CAP_CL21_SAM, F.Cu at (105.5, 109.7)
- added C7: 4.7uF, CL10A475KP8NNNC:CAP_0603_CL10A_1P6XP8_SAM, F.Cu at (98.0, 124.0)
- added C8: 0.1uF, CL10B104KB8NNNC:CAP_CL10_SAM, F.Cu at (123.4, 104.2)
- added C9: 10uF, CL21A106KOQNNNE:CAP_CL21_SAM, F.Cu at (123.3, 102.5)
- added Kailh_Switch3: Thumb1, Kailh_Switch:Kailh_Switch, F.Cu at (95.0, 85.0)
- added Kailh_Switch4: Thumb2, Kailh_Switch:Kailh_Switch, F.Cu at (95.0, 98.5)
- added L1: 470nH, CIGT201610EHR47MNE:RES_CIGT201610, F.Cu at (100.9, 117.3)
- added R1: 10k, RC1005F103CS:RES_1005_SAM, F.Cu at (123.1, 111.5)
- added R2: 13, RC0805FR_0713RL:RC0805N_YAG, F.Cu at (123.4, 106.0)
- added R3: 220k, RMCF0603FT220K:STA_RMCF0603_STP, F.Cu at (103.9, 116.4)
- added R4: 100k, RC0402FR_07100KL:RC0402N_YAG, F.Cu at (103.9, 118.0)
- added SW1: Power, EG1218:SW_1218_EWI, B.Cu at (128.2, 127.6)
- added SW2: Signal, EG1218:SW_1218_EWI, B.Cu at (128.2, 122.0)
- added SW3: Scroll_Button, 1825910-6:SW4_1825910-B_TEC, F.Cu at (130.0, 70.8)
- added SW4: DPI_Button, 1825910-6:SW4_1825910-B_TEC, F.Cu at (112.7, 96.5)
- added U1: DLC0008A, TPS62821DLCR:TPS62821DLCR, F.Cu at (100.7, 121.9)
- added U2: TTC_Gold_Encoder, TTC_Gold_Encoder:TTC_Gold_Encoder, F.Cu at (101.5, 74.0)
- Kailh_Switch1: value ~ -> Left
- Kailh_Switch2: value ~ -> Right
- NRF52840_ProMicro1: value ~ -> nrf52840
- PMW3389DM-T3QU1: value ~ -> pmw3389
- moved Kailh_Switch1 47.9 mm to (100.0, 60.0)
- moved J1 43.1 mm to (130.7, 115.0), turned to 180 degrees
- moved PMW3389DM-T3QU1 39.7 mm to (115.0, 110.0)
- moved NRF52840_ProMicro1 35.0 mm to (115.0, 66.5)
- moved Kailh_Switch2 26.7 mm to (130.0, 60.0)
Connections:
- J1 pad 1: unconnected-(J1-Pad1) -> GND
- J1 pad 2: unconnected-(J1-Pad2) -> BATT 3.7V
- Kailh_Switch1 pad 2: Net-(Kailh_Switch1-NO) -> Left
- Kailh_Switch2 pad 2: Net-(Kailh_Switch2-NO) -> Right
- NRF52840_ProMicro1 pad 1: (no net) -> GND
- NRF52840_ProMicro1 pad 10: (no net) -> Encoder_B
- NRF52840_ProMicro1 pad 11: (no net) -> 2.4 GHz
- NRF52840_ProMicro1 pad 12: (no net) -> BlueTooth
- NRF52840_ProMicro1 pad 13: (no net) -> NRESET
- NRF52840_ProMicro1 pad 14: (no net) -> SCLK
- NRF52840_ProMicro1 pad 15: (no net) -> MOTION
- NRF52840_ProMicro1 pad 16: (no net) -> MOSI
- NRF52840_ProMicro1 pad 17: (no net) -> MISO
- NRF52840_ProMicro1 pad 18: (no net) -> NCS
- NRF52840_ProMicro1 pad 19: (no net) -> DPI_Button
- NRF52840_ProMicro1 pad 2: (no net) -> unconnected-(NRF52840_ProMicro1-D1-Pad2)
- NRF52840_ProMicro1 pad 20: (no net) -> Scroll_Button
- NRF52840_ProMicro1 pad 21: (no net) -> Right
- NRF52840_ProMicro1 pad 22: (no net) -> VDD 3.3V
- NRF52840_ProMicro1 pad 23: (no net) -> unconnected-(NRF52840_ProMicro1-Reset-Pad23)
- NRF52840_ProMicro1 pad 24: (no net) -> GND
- NRF52840_ProMicro1 pad 25: (no net) -> unconnected-(NRF52840_ProMicro1-Battery+-Pad25)
- NRF52840_ProMicro1 pad 26: (no net) -> BATT 3.7V
- NRF52840_ProMicro1 pad 3: (no net) -> Left
- NRF52840_ProMicro1 pad 4: (no net) -> unconnected-(NRF52840_ProMicro1-GND-Pad4)
- NRF52840_ProMicro1 pad 5: (no net) -> unconnected-(NRF52840_ProMicro1-GND-Pad5)
- NRF52840_ProMicro1 pad 6: (no net) -> Thumb_1
- NRF52840_ProMicro1 pad 7: (no net) -> Thumb_2
- NRF52840_ProMicro1 pad 8: (no net) -> unconnected-(NRF52840_ProMicro1-D4-Pad8)
- NRF52840_ProMicro1 pad 9: (no net) -> Encoder_A
- PMW3389DM-T3QU1 pad 10: /SCLK -> SCLK
- PMW3389DM-T3QU1 pad 11: /MOSI -> MOSI
- PMW3389DM-T3QU1 pad 13: /NCS -> NCS
- PMW3389DM-T3QU1 pad 7: unconnected-(PMW3389DM-T3QU1-NRESET-Pad7) -> NRESET
- PMW3389DM-T3QU1 pad 9: /MOTION -> MOTION
Routing:
- net VDD 3.3V: track 0.00 -> 96.1 mm
- net BATT 3.7V: track 0.00 -> 81.4 mm
- net VDD 1.9V: track 0.00 -> 63.3 mm
- net 2.4 GHz: track 0.00 -> 57.3 mm
- net BlueTooth: track 0.00 -> 53.7 mm
- net Thumb_2: track 0.00 -> 41.5 mm
- net MISO: track 0.00 -> 41.5 mm
- net NCS: track 0.00 -> 40.2 mm
- net MOTION: track 0.00 -> 39.8 mm
- net NRESET: track 0.00 -> 39.2 mm
- net MOSI: track 0.00 -> 38.5 mm
- net SCLK: track 0.00 -> 35.2 mm
- net VCC 3.7V: track 0.00 -> 34.5 mm
- net DPI_Button: track 0.00 -> 31.6 mm
- net Thumb_1: track 0.00 -> 29.5 mm
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- added copper zone on B.Cu, net GND
- added copper zone on F.Cu, net GND
Other:
- board outline added: 50 x 82 mm
