File: KiCad/Mouse_Project.kicad_pcb (KiCad board)
At the start: 2 copper layers, 50 x 82 mm, 35 parts, among them J1 B2B-PH-K-S, SW1 Power, SW2 Signal, SW3 Scroll_Button, SW4 DPI_Button, U1 DLC0008A, U2 TTC_Gold_Encoder

Commit message: Completed version 0.1
Parts:
- removed C12, C13, C14, C15, C16, C17: 0.1uF, CL10B104KB8NNNC:CAP_CL10_SAM
- removed R3: 220k, RMCF0603FT220K:STA_RMCF0603_STP
- removed R4: 100k, RC0402FR_07100KL:RC0402N_YAG
- added R5: CRGCQ1206F330K, CRGCQ1206F330K:RES_CRGCQ1206F330K_TEC, F.Cu at (104.8, 116.5)
- U1: value DLC0008A -> TPS62821DLCR
Connections:
- NRF52840_ProMicro1 pad 14: SCLK -> MISO
- NRF52840_ProMicro1 pad 15: MOTION -> MOSI
- NRF52840_ProMicro1 pad 16: MOSI -> SCLK
- NRF52840_ProMicro1 pad 17: MISO -> MOTION
Routing:
- net MOTION: track 39.8 -> 49.6 mm
- net MISO: track 41.5 -> 33.7 mm
- net SCLK: track 35.2 -> 42.4 mm
- net VDD 1.9V: track 63.3 -> 68.4 mm
- net Right: track 11.2 -> 8.99 mm
- net Left: track 11.1 -> 8.87 mm
- net Thumb_1: track 29.5 -> 27.2 mm
- net BlueTooth: track 53.7 -> 55.8 mm
- net DPI_Button: track 31.6 -> 29.7 mm
- net Thumb_2: track 41.5 -> 39.7 mm
- net Net-(R3-Pad2): track 1.68 -> 0.00 mm
- net MOSI: track 38.5 -> 36.9 mm
- net NRESET: track 39.2 -> 40.8 mm
Other:
- board text added: "2.4_GHz"
- board text added: "BATT"
- board text added: "BlueTooth"
- board text added: "V-0.1"
- board text added: "VCC"

Commit message: PCB v0.2 almost done
Parts:
- C1, C11, C6, C9: footprint CL21A106KOQNNNE:CAP_CL21_SAM -> CL31A106KBHNNNE:CL31A106KBHNNNE
- C10: footprint GRM0335C1H121JA01D:G-033_MUR -> C0805C121J5GACTU:C0805C121J5GACTU
- C2: value 4.7uF/10V -> 4.7uF; footprint CL10A475KP8NNNC:CAP_0603_CL10A_1P6XP8_SAM -> CL31B475KBHNNNE:CL31B475KBHNNNE
- C3, C4, C5, C8: footprint CL10B104KB8NNNC:CAP_CL10_SAM -> C1206C104K5RACTU:C1206C104K5RACTU
- C7: footprint CL10A475KP8NNNC:CAP_0603_CL10A_1P6XP8_SAM -> CL31B475KBHNNNE:CL31B475KBHNNNE
- L1: footprint CIGT201610EHR47MNE:RES_CIGT201610 -> DFE252012P-R47M=P2:DFE252012P-1R0M=P2
- R1: footprint RC1005F103CS:RES_1005_SAM -> RC1206FR_0710KL:RC1206FR-0710KL
- R5: value CRGCQ1206F330K -> 330k
- moved SW1 15.6 mm to (132.0, 112.5)
- moved SW2 15.0 mm to (132.0, 107.5)
- moved C10 13.8 mm to (100.5, 110.5), turned to 0 degrees
- moved C11 9.20 mm to (98.0, 108.0), turned to 180 degrees
- moved U1 9.16 mm to (103.0, 113.0), turned to -90 degrees
- moved C7 8.16 mm to (104.0, 118.5), turned to -90 degrees
- moved R5 7.63 mm to (98.0, 113.0), turned to 180 degrees
- moved J1 5.01 mm to (130.5, 120.0)
- moved C6 3.33 mm to (104.5, 106.5), turned to 90 degrees
- moved C5 3.01 mm to (107.0, 106.5), turned to 90 degrees
- moved C9 1.65 mm to (124.0, 101.0)
- moved C1 1.36 mm to (104.5, 110.5), turned to 90 degrees
- moved L1 1.35 mm to (100.5, 116.0), turned to 180 degrees
- moved C2 1.26 mm to (104.5, 105.5), turned to -90 degrees
- moved R2 1.15 mm to (124.5, 106.0)
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Connections:
- net BlueTooth renamed Bluetooth
- SW2 pad 1: GND -> 2.4 GHz
- SW2 pad 2: 2.4 GHz -> GND
Routing:
- net VDD 1.9V: track 68.4 -> 57.4 mm
- net Bluetooth: track 55.8 -> 46.5 mm
- net 2.4 GHz: track 57.7 -> 48.7 mm
- net VDD 3.3V: track 95.7 -> 103.6 mm
- net BATT 3.7V: track 81.4 -> 77.0 mm
- net VCC 3.7V: track 34.5 -> 38.8 mm
- net NRESET: track 40.8 -> 43.5 mm
- net Net-(PMW3389DM-T3QU1-VDDPIX): track 4.16 -> 6.57 mm
- net GND: track 4.53 -> 2.94 mm
- net Net-(U1-FB): track 1.85 -> 3.20 mm
- net Net-(PMW3389DM-T3QU1-LED1_P): track 2.19 -> 3.34 mm
Other:
- board size 50 x 82 mm -> 50 x 73 mm
- board text added: "Bluetooth"
- board text added: "V-0.2"
- board text removed: "BlueTooth"
- board text removed: "V-0.1"

Commit message: Completed v0.2
Ordered new PCB and components
Routing:
- net Bluetooth: track 46.5 -> 47.5 mm
- net 2.4 GHz: track 48.7 -> 49.7 mm
Changed lines of the file:
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@@
 			(layer "Cmts.User")
 		)
-		(fp_rect
-			(start -5.4 -3.05)
+		(fp_line
+			(start -5.4 -0.95)
 			(end -3.6 -0.95)
 			(stroke
@@
 				(type default)
 			)
-			(fill yes)
 			(layer "Edge.Cuts")
 		)
-		(fp_rect
+		(fp_line
+			(start -5.4 -0.95)
+			(end -5.4 -3.05)
+			(stroke
+				(width 0.05)
+				(type default)
+			)
+			(layer "Edge.Cuts")
+		)
+		(fp_line
+			(start 3.6 -0.95)
+			(end 5.4 -0.95)
+			(stroke
+				(width 0.05)
+				(type default)
+			)
+			(layer "Edge.Cuts")
+		)
+		(fp_line
+			(start 3.6 -0.95)
+			(end 3.6 -3.05)
+			(stroke
+				(width 0.05)
+				(type default)
+			)
+			(layer "Edge.Cuts")
+		)
+		(fp_line
+			(start -3.6 -3.05)
+			(end -3.6 -0.95)
+			(stroke
+				(width 0.05)
+				(type default)
+			)
+			(layer "Edge.Cuts")
+		)
+		(fp_line
+			(start -3.6 -3.05)
+			(end -5.4 -3.05)
+			(stroke
+				(width 0.05)
+				(type default)
+			)
+			(layer "Edge.Cuts")
+		)
+		(fp_line
 			(start 5.4 -3.05)
-			(end 3.6 -0.95)
+			(end 5.4 -0.95)
+			(stroke
+				(width 0.05)
+				(type default)
+			)
+			(layer "Edge.Cuts")
+		)
+		(fp_line
+			(start 5.4 -3.05)
+			(end 3.6 -3.05)
 			(stroke
 				(width 0.05)
 				(type default)
 			)
-			(fill yes)
 			(layer "Edge.Cuts")
 		)
@@
 	)
 	(segment
-		(start 109.25 78.56666)
-		(end 109.25 89)
+		(start 124 92.5)
+		(end 134.5 103)
 		(width 0.5)
 		(layer "F.Cu")
@@
 	)
 	(segment
-		(start 124.5 93)
-		(end 134.5 103)
+		(start 134.5 103)
+		(end 134.5 107.5)
 		(width 0.5)
 		(layer "F.Cu")
@@
 	)
 	(segment
-		(start 109.25 89)
-		(end 113.25 93)
+		(start 109.25 90.75)
+		(end 111 92.5)
 		(width 0.5)
 		(layer "F.Cu")
@@
 	)
 	(segment
-		(start 134.5 103)
-		(end 134.5 107.5)
+		(start 111 92.5)
+		(end 124 92.5)
 		(width 0.5)
 		(layer "F.Cu")
@@
 	)
 	(segment
-		(start 113.25 93)
-		(end 124.5 93)
+		(start 107.35 76.66666)
+		(end 109.25 78.56666)
 		(width 0.5)
 		(layer "F.Cu")
@@
 	)
 	(segment
-		(start 107.35 76.66666)
-		(end 109.25 78.56666)
+		(start 109.25 78.56666)
+		(end 109.25 90.75)
 		(width 0.5)
 		(layer "F.Cu")
@@
 	)
 	(segment
-		(start 124 94.5)
-		(end 129.5 100)
+		(start 129.5 100)
+		(end 129.5 107.5)
 		(width 0.5)
 		(layer "F.Cu")
@@
 	)
 	(segment
-		(start 129.5 100)
-		(end 129.5 107.5)
+		(start 107.35 79.208326)
+		(end 106.570837 79.208326)
 		(width 0.5)
 		(layer "F.Cu")
@@
 	)
 	(segment
-		(start 106.570837 79.208326)
-		(end 105 80.779163)
+		(start 110.5 94)
+		(end 123.5 94)
 		(width 0.5)
 		(layer "F.Cu")
@@
 	)
 	(segment
-		(start 112.75 94.5)
-		(end 124 94.5)
+		(start 123.5 94)
+		(end 129.5 100)
 		(width 0.5)
 		(layer "F.Cu")
@@
 	)
 	(segment
-		(start 107.35 79.208326)
-		(end 106.570837 79.208326)
+		(start 106.570837 79.208326)
+		(end 105 80.779163)
 		(width 0.5)
 		(layer "F.Cu")
@@
 	(segment
 		(start 105 80.779163)
-		(end 105 86.75)
+		(end 105 88.5)
 		(width 0.5)
 		(layer "F.Cu")
@@
 	)
 	(segment
-		(start 105 86.75)
-		(end 112.75 94.5)
+		(start 105 88.5)
+		(end 110.5 94)
 		(width 0.5)
 		(layer "F.Cu")
