File: KiCad/Mouse_Project.kicad_sch (KiCad schematic)
At the start: 21 parts, among them U1 TPS62821DLCR

Commit message: backup
Parts:
- added J1: B2B-PH-K-S, B2B-PH-K-S:CONN2_B2B-PH-K-S_JST, symbol B2B-PH-K-S:B2B-PH-K-S
- added J2: B2B-PH-K-S_simple, B2B-PH-K-S:CONN2_B2B-PH-K-S_JST, symbol B2B-PH-K-S:B2B-PH-K-S_simple
- C10: value C -> optional
- C11: value C -> 10uF
- C9: value C -> 4.7uF
- L1: value L -> 470nH
- NRF52840_ProMicro1: footprint NRF52840_ProMicro -> nrf52840_promicro:nrf52840_promicro
Changed lines of the file:
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@@
 			)
 		)
-		(property "Value" "C"
+		(property "Value" "optional"
 			(at 287.02 266.6999 0)
 			(effects
@@
 			)
 		)
-		(property "Footprint" "NRF52840_ProMicro"
+		(property "Footprint" "nrf52840_promicro:nrf52840_promicro"
 			(at 303.53 211.836 0)
 			(effects
@@
 	)
 	(symbol
+		(lib_id "B2B-PH-K-S:B2B-PH-K-S_simple")
+		(at 374.65 241.3 0)
+		(unit 1)
+		(exclude_from_sim no)
+		(in_bom yes)
+		(on_board yes)
+		(dnp no)
+		(fields_autoplaced yes)
+		(property "Reference" "J2"
+			(at 388.62 241.2999 0)
+			(effects
+				(font
+					(size 1.524 1.524)
+				)
+				(justify left)
+			)
+		)
+		(property "Value" "B2B-PH-K-S_simple"
+			(at 388.62 243.8399 0)
+			(effects
+				(font
+					(size 1.524 1.524)
+				)
+				(justify left)
+			)
+		)
+		(property "Footprint" "B2B-PH-K-S:CONN2_B2B-PH-K-S_JST"
+			(at 374.65 241.3 0)
+			(effects
+				(font
+					(size 1.27 1.27)
+					(italic yes)
+				)
+				(hide yes)
+			)
+		)
+		(property "Datasheet" "B2B-PH-K-S"
+			(at 374.65 241.3 0)
+			(effects
+				(font
+					(size 1.27 1.27)
+					(italic yes)
+				)
+				(hide yes)
+			)
+		)
+		(property "Description" ""
+			(at 374.65 241.3 0)
+			(effects
+				(font
+					(size 1.27 1.27)
+				)
+				(hide yes)
+			)
+		)
+		(pin "2"
+		)
+		(pin "1"
+		)
+		(instances
+			(project ""
+				(path "/0dfb68a1-d60c-4876-81e5-ddb5b2679ca1"
+					(reference "J2")
+					(unit 1)
+				)
+			)
+		)
+	)
+	(symbol
 		(lib_id "power:GND")
 		(at 139.7 161.29 0)
@@
 			)
 		)
-		(property "Value" "C"
+		(property "Value" "4.7uF"
 			(at 220.98 274.3199 0)
 			(effects
@@
 	)
 	(symbol
+		(lib_id "B2B-PH-K-S:B2B-PH-K-S")
+		(at 383.54 231.14 0)
+		(unit 1)
+		(exclude_from_sim no)
+		(in_bom yes)
+		(on_board yes)
+		(dnp no)
+		(fields_autoplaced yes)
+		(property "Reference" "J1"
+			(at 391.16 228.5999 0)
+			(effects
+				(font
+					(size 1.27 1.27)
+				)
+				(justify left)
+			)
+		)
+		(property "Value" "B2B-PH-K-S"
+			(at 391.16 231.1399 0)
+			(effects
+				(font
+					(size 1.27 1.27)
+				)
+				(justify left)
+			)
+		)
+		(property "Footprint" "B2B-PH-K-S:CONN2_B2B-PH-K-S_JST"
+			(at 383.54 231.14 0)
+			(effects
+				(font
+					(size 1.27 1.27)
+				)
+				(justify bottom)
+				(hide yes)
+			)
+		)
+		(property "Datasheet" ""
+			(at 383.54 231.14 0)
+			(effects
+				(font
+					(size 1.27 1.27)
+				)
+				(hide yes)
+			)
+		)
+		(property "Description" ""
+			(at 383.54 231.14 0)
+			(effects
+				(font
+					(size 1.27 1.27)
+				)
+				(hide yes)
+			)
+		)
+		(property "MANUFACTURER" "JST"
+			(at 383.54 231.14 0)
+			(effects
+				(font
+					(size 1.27 1.27)
+				)
+				(justify bottom)
+				(hide yes)
+			)
+		)
+		(pin "1"
+		)
+		(pin "2"
+		)
+		(instances
+			(project ""
+				(path "/0dfb68a1-d60c-4876-81e5-ddb5b2679ca1"
+					(reference "J1")
+					(unit 1)
+				)
+			)
+		)
+	)
+	(symbol
 		(lib_id "power:GND")
 		(at 386.08 146.05 0)
@@
 			)
 		)
-		(property "Value" "C"
+		(property "Value" "10uF"
 			(at 299.72 266.6999 0)
 			(effects
@@
 			)
 		)
-		(property "Value" "L"
+		(property "Value" "470nH"
 			(at 267.97 257.81 90)
 			(effects

Commit message: Almost done
Parts:
- removed J2: B2B-PH-K-S_simple, B2B-PH-K-S:CONN2_B2B-PH-K-S_JST, symbol B2B-PH-K-S:B2B-PH-K-S_simple
- added C12, C13, C14, C15, C16, C17: 0.1uF, CL10B104KB8NNNC:CAP_CL10_SAM, symbol Device:C
- added Kailh_Switch3: Thumb1, Kailh_Switch:Kailh_Switch, symbol Kailh_Switch:Kailh_Switch
- added Kailh_Switch4: Thumb2, Kailh_Switch:Kailh_Switch, symbol Kailh_Switch:Kailh_Switch
- added SW1: Power, SW_1218_EWI, symbol EG1218:EG1218
- added SW2: Signal, SW_1218_EWI, symbol EG1218:EG1218
- added SW3: Scroll_Button, 1825910-6:SW4_1825910-B_TEC, symbol 1825910-6:1825910-6
- added SW4: DPI_Button, 1825910-6:SW4_1825910-B_TEC, symbol 1825910-6:1825910-6
- added U2: TTC_Gold_Encoder, TTC_Gold_Encoder:TTC_Gold_Encoder, symbol TTC_Gold_Encoder:TTC_Gold_Encoder
- C1: renamed from C5; value C -> 10uF; footprint (none) -> CL21A106KOQNNNE:CAP_CL21_SAM
- C10: value optional -> 120pF; footprint (none) -> GRM0335C1H121JA01D:G-033_MUR
- C11: footprint (none) -> CL21A106KOQNNNE:CAP_CL21_SAM
- C2: renamed from C7; value C -> 4.7uF/10V; footprint (none) -> CL10A475KP8NNNC:CAP_0603_CL10A_1P6XP8_SAM
- C3: renamed from C6; value C -> 0.1uF; footprint (none) -> CL10B104KB8NNNC:CAP_CL10_SAM
- C4: renamed from C8; value C -> 0.1uF; footprint (none) -> CL10B104KB8NNNC:CAP_CL10_SAM
- C5: renamed from C4; value C -> 0.1uF; footprint (none) -> CL10B104KB8NNNC:CAP_CL10_SAM
- C6: renamed from C3; value C -> 10uF; footprint (none) -> CL21A106KOQNNNE:CAP_CL21_SAM
- C7: renamed from C9; footprint (none) -> CL10A475KP8NNNC:CAP_0603_CL10A_1P6XP8_SAM
- C8: renamed from C1; value C -> 0.1uF; footprint (none) -> CL10B104KB8NNNC:CAP_CL10_SAM
- C9: renamed from C2; value C -> 10uF; footprint (none) -> CL21A106KOQNNNE:CAP_CL21_SAM
- Kailh_Switch1: value ~ -> Left
- Kailh_Switch2: value ~ -> Right
- L1: footprint (none) -> CIGT201610EHR47MNE:RES_CIGT201610
- NRF52840_ProMicro1: value ~ -> nrf52840
- PMW3389DM-T3QU1: value ~ -> pmw3389
- R1: renamed from R2; value R -> 10k; footprint (none) -> RC1005F103CS:RES_1005_SAM
- R2: renamed from R1; value R -> 13; footprint (none) -> RC0805FR_0713RL:RC0805N_YAG
- R3: value R -> 220k; footprint (none) -> RMCF0603FT220K:STA_RMCF0603_STP
- R4: value R -> 100k; footprint (none) -> RC0402FR_07100KL:RC0402N_YAG
- U1: footprint DLC0008A -> TPS62821DLCR:TPS62821DLCR
Connections:
- net VDD - 1.9V is gone; now on net VDD 1.9V: C10.1, C11.1, L1.2, R3.1
- net GND: now also J1.1, NRF52840_ProMicro1.1 (GND), NRF52840_ProMicro1.24 (GND), C12.2, C13.2, C14.2, C15.2, C16.2, C17.2, Kailh_Switch3.1 (COM), Kailh_Switch4.1 (COM), SW2.1, SW3.3, SW3.4, SW4.3, SW4.4, U2.3 (Com); no longer NRF52840_ProMicro1.GND
- net MISO: now also NRF52840_ProMicro1.17 (D15)
- net MOSI: now also NRF52840_ProMicro1.16 (D14)
- net MOTION: now also NRF52840_ProMicro1.15 (D16)
- net NCS: now also NRF52840_ProMicro1.18 (D18)
- net SCLK: now also NRF52840_ProMicro1.14 (D10)
- net VDD 3.3V: now also NRF52840_ProMicro1.22 (3.3V); no longer NRF52840_ProMicro1.VCC (3.3V)
- net Right: now reaches Kailh_Switch2.2 (NO)
- net Right: now also NRF52840_ProMicro1.21 (D21), C15.1; no longer NRF52840_ProMicro1.002 (D19)
- net Left: now reaches Kailh_Switch1.2 (NO)
- net Left: now also NRF52840_ProMicro1.3 (D0), C14.1; no longer NRF52840_ProMicro1.029 (D20)
- net BATT 3.7V: now reaches J1.2
- net BATT 3.7V: now also NRF52840_ProMicro1.26 (Battery+), SW1.1
- net NRESET: now reaches PMW3389DM-T3QU1.7 (NRESET)
- net NRESET: now also NRF52840_ProMicro1.13 (D9)
- net VCC - 3.7V renamed VCC 3.7V
- net VCC 3.7V: now also SW1.2
- new net 2.4 GHz: NRF52840_ProMicro1.11 (D7), SW2.2
- new net BlueTooth: NRF52840_ProMicro1.12 (D8), SW2.3
- new net DPI_Button: C13.1, NRF52840_ProMicro1.19 (D19), SW4.1, SW4.2
- new net Encoder_A: NRF52840_ProMicro1.9 (D5), U2.1 (A)
- new net Encoder_B: NRF52840_ProMicro1.10 (D6), U2.2 (B)
- new net Scroll_Button: C12.1, NRF52840_ProMicro1.20 (D20), SW3.1, SW3.2
- new net Thumb_1: C16.1, Kailh_Switch3.2 (NO), NRF52840_ProMicro1.6 (D2)
- new net Thumb_2: C17.1, Kailh_Switch4.2 (NO), NRF52840_ProMicro1.7 (D3)
- no-connect marks 3 -> 8
Other:
- note added: "3.7V LiPO JST"
- note added: "Bottom Switches"
- note added: "Scroll Wheel"
- moved on the sheet: C1, C10, C11, C2, C3, C4, C5, C6, C7, C8, C9, J1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

Commit message: Completed version 0.1
Parts:
- removed C12, C13, C14, C15, C16, C17: 0.1uF, CL10B104KB8NNNC:CAP_CL10_SAM, symbol Device:C
- removed R3: 220k, RMCF0603FT220K:STA_RMCF0603_STP, symbol Device:R
- removed R4: 100k, RC0402FR_07100KL:RC0402N_YAG, symbol Device:R
- added R5: 330k, RES_CRGCQ1206F330K_TEC, symbol CRGCQ1206F330K:CRGCQ1206F330K
Connections:
- net GND: now also R5.2
- net MISO: now also NRF52840_ProMicro1.14 (D10); no longer NRF52840_ProMicro1.17 (D15)
- net MOSI: now also NRF52840_ProMicro1.15 (D16); no longer NRF52840_ProMicro1.16 (D14)
- net MOTION: now also NRF52840_ProMicro1.17 (D15); no longer NRF52840_ProMicro1.15 (D16)
- net SCLK: now also NRF52840_ProMicro1.16 (D14); no longer NRF52840_ProMicro1.14 (D10)
- net VDD 1.9V: now also R5.1

Commit message: PCB v0.2 almost done
Parts:
- C1, C11, C6, C9: footprint CL21A106KOQNNNE:CAP_CL21_SAM -> CL31A106KBHNNNE:CL31A106KBHNNNE
- C10: footprint GRM0335C1H121JA01D:G-033_MUR -> C0805C121J5GACTU:C0805C121J5GACTU
- C2: value 4.7uF/10V -> 4.7uF; footprint CL10A475KP8NNNC:CAP_0603_CL10A_1P6XP8_SAM -> CL31B475KBHNNNE:CL31B475KBHNNNE
- C3, C4, C5, C8: footprint CL10B104KB8NNNC:CAP_CL10_SAM -> C1206C104K5RACTU:C1206C104K5RACTU
- C7: footprint CL10A475KP8NNNC:CAP_0603_CL10A_1P6XP8_SAM -> CL31B475KBHNNNE:CL31B475KBHNNNE
- L1: footprint CIGT201610EHR47MNE:RES_CIGT201610 -> DFE252012P-R47M=P2:DFE252012P-1R0M=P2
- R1: footprint RC1005F103CS:RES_1005_SAM -> RC1206FR_0710KL:RC1206FR-0710KL
Connections:
- net 2.4 GHz: now also SW2.1; no longer SW2.2
- net GND: now also SW2.2; no longer SW2.1
- net BlueTooth renamed Bluetooth
